File: eagle/DJ CONTROLLER.sch (EAGLE design)
At the start: 91 parts, among them IC1 74HC4051, IC2 74HC4051, IC3 74HC4051, IC4 74HC4051

Commit message: Add files via upload
Parts:
- added JP79: (no value), pinhead:PINHD-1X2
Connections:
- new net N$43: B1.RESET, JP79.2
- net GND: now also JP79.1
Changed lines of the file:
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@@
 <part name="GND8" library="supply1" deviceset="AGND" device="" value="GND"/>
 <part name="P+8" library="supply1" deviceset="+5V" device=""/>
+<part name="JP79" library="pinhead" deviceset="PINHD-1X2" device=""/>
 </parts>
 <sheets>
@@
 <instance part="JP78" gate="G$1" x="713.74" y="40.64" rot="R90"/>
 <instance part="GND7" gate="VR1" x="678.18" y="0"/>
-<instance part="GND8" gate="VR1" x="55.88" y="142.24"/>
+<instance part="GND8" gate="VR1" x="17.78" y="124.46"/>
 <instance part="P+8" gate="1" x="55.88" y="175.26" rot="R90"/>
+<instance part="JP79" gate="G$1" x="38.1" y="144.78" rot="R180"/>
 </instances>
 <busses>
@@
 <wire x1="63.5" y1="152.4" x2="63.5" y2="149.86" width="0.1524" layer="91"/>
 <wire x1="63.5" y1="149.86" x2="73.66" y2="149.86" width="0.1524" layer="91"/>
-<wire x1="73.66" y1="149.86" x2="55.88" y2="149.86" width="0.1524" layer="91"/>
-<wire x1="55.88" y1="149.86" x2="55.88" y2="144.78" width="0.1524" layer="91"/>
+<wire x1="73.66" y1="149.86" x2="17.78" y2="149.86" width="0.1524" layer="91"/>
+<wire x1="17.78" y1="149.86" x2="17.78" y2="134.62" width="0.1524" layer="91"/>
 <pinref part="GND8" gate="VR1" pin="AGND"/>
+<pinref part="JP79" gate="G$1" pin="1"/>
+<wire x1="17.78" y1="134.62" x2="17.78" y2="127" width="0.1524" layer="91"/>
+<wire x1="40.64" y1="142.24" x2="48.26" y2="142.24" width="0.1524" layer="91"/>
+<wire x1="48.26" y1="142.24" x2="48.26" y2="134.62" width="0.1524" layer="91"/>
+<wire x1="48.26" y1="134.62" x2="17.78" y2="134.62" width="0.1524" layer="91"/>
 </segment>
 </net>
@@
 </segment>
 </net>
-<net name="N$1" class="0">
+<net name="SS" class="0">
 <segment>
 <wire x1="373.38" y1="276.86" x2="607.06" y2="276.86" width="0.1524" layer="91"/>
@@
 </segment>
 </net>
+<net name="N$43" class="0">
+<segment>
+<pinref part="JP79" gate="G$1" pin="2"/>
+<pinref part="B1" gate="BOARD" pin="RESET"/>
+<wire x1="40.64" y1="144.78" x2="73.66" y2="144.78" width="0.1524" layer="91"/>
+</segment>
+</net>

Commit message: added noise reduction capacitors for analog inputs
Parts:
- added C1, C2, C3, C4, C5, C6: (no value), resistor:C-EU050-025X075
Connections:
- net FAD1: now also C4.1
- net FAD2: now also C3.1
- net FAD3: now also C2.1
- net FAD4: now also C1.1
- net GND: now also C1.2, C2.2, C3.2, C4.2, C5.2, C6.2
- net MODE1: now also C5.1
- net MODE2: now also C6.1
